File: SerialOptoConnect.kicad_sch (KiCad schematic)
At the start: 20 parts, among them J1 Conn_01x06_Pin, J2 Conn_01x10_Pin, Q1 BC547, Q2 BC547, U1 PC817, U2 PC817, U3 PC817, U4 PC817

Commit message: some small alignments
Parts:
- removed R10, R5: 1k, Resistor_THT:R_Axial_DIN0204_L3.6mm_D1.6mm_P5.08mm_Horizontal, symbol Device:R
- R4, R9: value 1k -> 10k
Other:
- moved on the sheet: R4
Changed lines of the file:
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@@
-	)
-	(junction
-		(at 85.09 68.58)
-		(diameter 0)
-		(color 0 0 0 0)
 	)
 	(junction
@@
 	)
 	(junction
-		(at 39.37 124.46)
-		(diameter 0)
-		(color 0 0 0 0)
-	)
-	(junction
 		(at 91.44 123.19)
 		(diameter 0)
@@
 	(wire
 		(pts
-			(xy 85.09 58.42) (xy 85.09 59.69)
-		)
-		(stroke
-			(width 0)
-			(type default)
-		)
-	)
-	(wire
-		(pts
 			(xy 39.37 95.25) (xy 39.37 97.79)
 		)
@@
 	(wire
 		(pts
+			(xy 85.09 53.34) (xy 85.09 58.42)
+		)
+		(stroke
+			(width 0)
+			(type default)
+		)
+	)
+	(wire
+		(pts
 			(xy 71.12 101.6) (xy 71.12 107.95)
 		)
@@
 	(wire
 		(pts
-			(xy 85.09 50.8) (xy 85.09 40.64)
+			(xy 85.09 45.72) (xy 85.09 40.64)
 		)
 		(stroke
@@
 	(wire
 		(pts
-			(xy 39.37 109.22) (xy 39.37 113.03)
-		)
-		(stroke
-			(width 0)
-			(type default)
-		)
-	)
-	(wire
-		(pts
 			(xy 44.45 101.6) (xy 44.45 109.22)
 		)
@@
 	(wire
 		(pts
-			(xy 39.37 124.46) (xy 39.37 125.73)
-		)
-		(stroke
-			(width 0)
-			(type default)
-		)
-	)
-	(wire
-		(pts
 			(xy 97.79 123.19) (xy 91.44 123.19)
 		)
@@
 	(wire
 		(pts
-			(xy 39.37 124.46) (xy 41.91 124.46)
-		)
-		(stroke
-			(width 0)
-			(type default)
-		)
-	)
-	(wire
-		(pts
 			(xy 63.5 100.33) (xy 63.5 111.76)
 		)
@@
 	(wire
 		(pts
-			(xy 41.91 106.68) (xy 41.91 124.46)
+			(xy 41.91 106.68) (xy 41.91 125.73)
 		)
 		(stroke
@@
 	(wire
 		(pts
-			(xy 85.09 68.58) (xy 80.01 68.58)
-		)
-		(stroke
-			(width 0)
-			(type default)
-		)
-	)
-	(wire
-		(pts
 			(xy 85.09 40.64) (xy 82.55 40.64)
 		)
@@
 	(wire
 		(pts
-			(xy 39.37 120.65) (xy 39.37 124.46)
-		)
-		(stroke
-			(width 0)
-			(type default)
-		)
-	)
-	(wire
-		(pts
 			(xy 80.01 68.58) (xy 78.74 68.58)
 		)
@@
 	(wire
 		(pts
-			(xy 85.09 67.31) (xy 85.09 68.58)
-		)
-		(stroke
-			(width 0)
-			(type default)
-		)
-	)
-	(wire
-		(pts
 			(xy 63.5 91.44) (xy 63.5 92.71)
 		)
@@
 	(wire
 		(pts
-			(xy 85.09 68.58) (xy 110.49 68.58)
+			(xy 80.01 68.58) (xy 110.49 68.58)
 		)
 		(stroke
@@
 	(symbol
 		(lib_id "power:GND")
-		(at 39.37 125.73 0)
+		(at 41.91 125.73 0)
 		(unit 1)
 		(exclude_from_sim no)
@@
 		(fields_autoplaced yes)
 		(property "Reference" "#PWR08"
-			(at 39.37 132.08 0)
+			(at 41.91 132.08 0)
 			(effects
 				(font
@@
 		)
 		(property "Value" "GND"
-			(at 39.37 130.81 0)
+			(at 41.91 130.81 0)
 			(effects
 				(font
@@
 		)
 		(property "Footprint" ""
-			(at 39.37 125.73 0)
+			(at 41.91 125.73 0)
 			(effects
 				(font
@@
 		)
 		(property "Datasheet" ""
-			(at 39.37 125.73 0)
+			(at 41.91 125.73 0)
 			(effects
 				(font
@@
 		)
 		(property "Description" "Power symbol creates a global label with name \"GND\" , ground"
-			(at 39.37 125.73 0)
+			(at 41.91 125.73 0)
 			(effects
 				(font
@@
 			)
 		)
-		(property "Value" "1k"
+		(property "Value" "10k"
 			(at 41.91 102.8699 0)
 			(effects
@@
 	)
 	(symbol
-		(lib_id "Device:R")
-		(at 85.09 63.5 0)
-		(unit 1)
-		(exclude_from_sim no)
-		(in_bom yes)
-		(on_board yes)
-		(dnp no)
-		(fields_autoplaced yes)
-		(property "Reference" "R5"
-			(at 87.63 62.2299 0)
-			(effects
-				(font
-					(size 1.27 1.27)
-				)
-				(justify left)
-			)
-		)
-		(property "Value" "1k"
-			(at 87.63 64.7699 0)
-			(effects
-				(font
-					(size 1.27 1.27)
-				)
-				(justify left)
-			)
-		)
-		(property "Footprint" "Resistor_THT:R_Axial_DIN0204_L3.6mm_D1.6mm_P5.08mm_Horizontal"
-			(at 83.312 63.5 90)
-			(effects
-				(font
-					(size 1.27 1.27)
-				)
-				(hide yes)
-			)
-		)
-		(property "Datasheet" "~"
-			(at 85.09 63.5 0)
-			(effects
-				(font
-					(size 1.27 1.27)
-				)
-				(hide yes)
-			)
-		)
-		(property "Description" "Resistor"
-			(at 85.09 63.5 0)
-			(effects
-				(font
-					(size 1.27 1.27)
-				)
-				(hide yes)
-			)
-		)
-		(pin "2"
-		)
-		(pin "1"
-		)
-		(instances
-			(project "SerialOptoConnect"
-				(path "/6aa56471-e065-4edd-8c70-ddc11bc1dc24"
-					(reference "R5")
-					(unit 1)
-				)
-			)
-		)
-	)
-	(symbol
 		(lib_id "Diode:1N5819")
 		(at 71.12 111.76 90)
@@
 	(symbol
 		(lib_id "Device:R")
-		(at 85.09 54.61 0)
+		(at 85.09 49.53 0)
 		(unit 1)
 		(exclude_from_sim no)
@@
 		(fields_autoplaced yes)
 		(property "Reference" "R4"
-			(at 87.63 53.3399 0)
+			(at 87.63 48.2599 0)
 			(effects
 				(font
@@
 			)
 		)
-		(property "Value" "1k"
-			(at 87.63 55.8799 0)
+		(property "Value" "10k"
+			(at 87.63 50.7999 0)
 			(effects
 				(font
@@
 		)
 		(property "Footprint" "Resistor_THT:R_Axial_DIN0204_L3.6mm_D1.6mm_P5.08mm_Horizontal"
-			(at 83.312 54.61 90)
+			(at 83.312 49.53 90)
 			(effects
 				(font
@@
 		)
 		(property "Datasheet" "~"
-			(at 85.09 54.61 0)
+			(at 85.09 49.53 0)
 			(effects
 				(font
@@
 		)
 		(property "Description" "Resistor"
-			(at 85.09 54.61 0)
+			(at 85.09 49.53 0)
 			(effects
 				(font
@@
 					(unit 1)
 				)
-			)
-		)
-	)
-	(symbol
-		(lib_id "Device:R")
-		(at 39.37 116.84 0)
-		(unit 1)
-		(exclude_from_sim no)
-		(in_bom yes)
-		(on_board yes)
-		(dnp no)
-		(fields_autoplaced yes)
-		(property "Reference" "R10"
-			(at 41.91 115.5699 0)
-			(effects
-				(font
-					(size 1.27 1.27)
-				)
-				(justify left)
-			)
-		)
-		(property "Value" "1k"
-			(at 41.91 118.1099 0)
-			(effects
-				(font
-					(size 1.27 1.27)
-				)
-				(justify left)
-			)
-		)
-		(property "Footprint" "Resistor_THT:R_Axial_DIN0204_L3.6mm_D1.6mm_P5.08mm_Horizontal"
-			(at 37.592 116.84 90)
-			(effects
-				(font
-					(size 1.27 1.27)
-				)
-				(hide yes)
-			)
-		)
-		(property "Datasheet" "~"
-			(at 39.37 116.84 0)
-			(effects
-				(font
-					(size 1.27 1.27)
-				)
-				(hide yes)
-			)
-		)
-		(property "Description" "Resistor"
-			(at 39.37 116.84 0)
-			(effects
-				(font
-					(size 1.27 1.27)
-				)
-				(hide yes)
-			)
-		)
-		(pin "2"
-		)
-		(pin "1"
-		)
-		(instances
-			(project "SerialOptoConnect"
-				(path "/6aa56471-e065-4edd-8c70-ddc11bc1dc24"
-					(reference "R10")
-					(unit 1)
-				)
